Commit message: onto path validation rbprm

File: data/urdf/box.urdf (robot description, URDF)
Before this commit: robot box, 1 links, 0 joints
Links:
- link base_link: geometry collision mesh filename=package://hpp-rbprm-corba/meshes/box.stl; visual mesh filename=package://hpp-rbprm-corba/meshes/robot_box.stl

File: data/urdf/box_rom.urdf (robot description, URDF)
Before this commit: robot box, 1 links, 0 joints
Links:
- link base_link: geometry collision mesh filename=package://hpp-rbprm-corba/meshes/box_rom.stl; visual mesh filename=package://hpp-rbprm-corba/meshes/box_rom.stl
