Commit message: rbprm now working m...

File: data/urdf/scene.urdf (robot description, URDF)
Before this commit: robot scene, 1 links, 0 joints
Links:
- link base_link: geometry collision mesh filename=package://hpp-rbprm-corba/meshes/ground.stl; visual mesh filename=package:///../hpp-rbprm-corba/meshes/ground.stl
