Commit message: crawll back scenario

File: data/urdf/scene_wall.urdf (robot description, URDF)
Before this commit: robot box, 1 links, 0 joints
Links:
- link base_link: geometry collision mesh filename=package://hpp-rbprm-corba/meshes/ground_table.stl; visual mesh filename=package:///../hpp-rbprm-corba/meshes/ground_table.stl
