Commit message: hrp2 boxes

File: data/urdf/hrp2_trunk.urdf (robot description, URDF)
Before this commit: robot hrp2_rom, 1 links, 0 joints
Links:
- link base_link: geometry collision mesh filename=package://hpp-rbprm-corba/meshes/hrp2_trunk.stl; visual mesh filename=package://hpp-rbprm-corba/meshes/hrp2_trunk.stl

File: data/urdf/truck.urdf (robot description, URDF)
Before this commit: robot hrp2_rom, 1 links, 0 joints
Links:
- link base_link: geometry collision mesh filename=package://hpp-rbprm-corba/meshes/truck.stl; visual mesh filename=package:///../hpp-rbprm-corba/meshes/truck_vision.stl
