Commit message: stair

File: data/urdf/box_rom.urdf (robot description, URDF)
Before this commit: robot hrp2_rom, 1 links, 0 joints
Links:
- link base_link: geometry collision mesh filename=package://hpp-rbprm-corba/meshes/box_rom.stl; visual mesh filename=package://hpp-rbprm-corba/meshes/box_rom.stl

File: data/urdf/hrp2_rom.urdf (robot description, URDF)
Before this commit: robot hrp2_trunk, 1 links, 0 joints
Links:
- link base_link: geometry collision mesh filename=package://hpp-rbprm-corba/meshes/hrp2_rom.stl; visual mesh filename=package://hpp-rbprm-corba/meshes/hrp2_rom.stl
