Commit message: flexible trunk

File: data/urdf/hrp2_larm_rom.urdf (robot description, URDF)
Before this commit: robot hrp2_larm_rom, 1 links, 0 joints
Links:
- added link BODY
- added link CHEST_LINK0
- added link torso; collision mesh filename=package://hpp-rbprm-corba/meshes/hrp2_larm_rom.stl; visual mesh filename=package://hpp-rbprm-corba/meshes/hrp2_larm_rom.stl
- link base_link: geometry 
Joints:
- added joint CHEST_JOINT0: type revolute, parent BODY, child CHEST_LINK0, origin xyz=0.032 0 0.3507 rpy=0 0 0, axis 0 0 1, limit lower=-0.785398 upper=0.785398 effort=151.1 velocity=4.40217
- added joint CHEST_JOINT1: type revolute, parent CHEST_LINK0, child torso, origin xyz=0 0 0 rpy=0 0 0, axis 0 1 0, limit lower=-0.0872665 upper=1.0472 effort=278.9 velocity=2.3963
- added joint WAIST: type fixed, parent base_link, child BODY, origin xyz=0 0 0 rpy=0 0 0

File: data/urdf/hrp2_lleg_rom.urdf (robot description, URDF)
Before this commit: robot hrp2_lleg_rom, 1 links, 0 joints
Links:
- added link BODY; collision mesh filename=package://hpp-rbprm-corba/meshes/hrp2_lleg_rom.stl; visual mesh filename=package://hpp-rbprm-corba/meshes/hrp2_lleg_rom.stl
- added link CHEST_LINK0
- added link torso
- link base_link: geometry 
Joints:
- added joint CHEST_JOINT0: type revolute, parent BODY, child CHEST_LINK0, origin xyz=0.032 0 0.3507 rpy=0 0 0, axis 0 0 1, limit lower=-0.785398 upper=0.785398 effort=151.1 velocity=4.40217
- added joint CHEST_JOINT1: type revolute, parent CHEST_LINK0, child torso, origin xyz=0 0 0 rpy=0 0 0, axis 0 1 0, limit lower=-0.0872665 upper=1.0472 effort=278.9 velocity=2.3963
- added joint WAIST: type fixed, parent base_link, child BODY, origin xyz=0 0 0 rpy=0 0 0

File: data/urdf/hrp2_rarm_rom.urdf (robot description, URDF)
Before this commit: robot hrp2_rarm_rom, 1 links, 0 joints
Links:
- added link BODY
- added link CHEST_LINK0
- added link torso; collision mesh filename=package://hpp-rbprm-corba/meshes/hrp2_rarm_rom.stl; visual mesh filename=package://hpp-rbprm-corba/meshes/hrp2_rarm_rom.stl
- link base_link: geometry 
Joints:
- added joint CHEST_JOINT0: type revolute, parent BODY, child CHEST_LINK0, origin xyz=0.032 0 0.3507 rpy=0 0 0, axis 0 0 1, limit lower=-0.785398 upper=0.785398 effort=151.1 velocity=4.40217
- added joint CHEST_JOINT1: type revolute, parent CHEST_LINK0, child torso, origin xyz=0 0 0 rpy=0 0 0, axis 0 1 0, limit lower=-0.0872665 upper=1.0472 effort=278.9 velocity=2.3963
- added joint WAIST: type fixed, parent base_link, child BODY, origin xyz=0 0 0 rpy=0 0 0

File: data/urdf/hrp2_trunk_flexible.urdf (robot description, URDF)
Before this commit: robot hrp2_rleg_rom, 4 links, 3 joints
Links:
- link BODY: geometry collision mesh filename=package://hpp-rbprm-corba/meshes/hrp2_trunk_body.stl; visual mesh filename=package://hpp-rbprm-corba/meshes/hrp2_trunk_body.stl
- link torso: geometry collision mesh filename=package://hpp-rbprm-corba/meshes/hrp2_trunk_torso.stl; visual mesh filename=package://hpp-rbprm-corba/meshes/hrp2_trunk_torso.stl
