Commit message: stait for justin

File: data/urdf/stair_bauzil.urdf (robot description, URDF)
Before this commit: robot stair_bauzil, 1 links, 0 joints
Links:
- link base_link: geometry collision mesh filename=package://hpp-rbprm-corba/meshes/stair_bauzil_reduced.stl; visual mesh filename=package:///../hpp-rbprm-corba/meshes/stair_bauzil.stl
