Commit message: fixed hrp2 rom

File: data/urdf/darpa.urdf (robot description, URDF)
Before this commit: robot chair, 1 links, 0 joints
Links:
- link base_link: geometry collision mesh filename=package://hpp-rbprm-corba/meshes/darpareduced.stl; visual mesh filename=package://hpp-rbprm-corba/meshes/darpareduced.stl

File: data/urdf/groundcrouch.urdf (robot description, URDF)
Before this commit: robot chair, 1 links, 0 joints
Links:
- link base_link: geometry collision mesh filename=package://hpp-rbprm-corba/meshes/groundcrouch.stl; visual mesh filename=package://hpp-rbprm-corba/meshes/groundcrouch.stl

File: data/urdf/hrp2_trunk_flexible.urdf (robot description, URDF)
Before this commit: robot hrp2_trunk_flexible, 4 links, 3 joints
Links:
- link BODY: geometry collision mesh filename=package://hpp-rbprm-corba/meshes/hrp2_trunk_body.stl; visual mesh filename=package://hpp-rbprm-corba/meshes/hrp2_trunk_body.stl

File: data/urdf/scene_wall.urdf (robot description, URDF)
Before this commit: robot scene_wall, 1 links, 0 joints
Links:
- link base_link: geometry collision mesh filename=package://hpp-rbprm-corba/meshes/ground_table.stl; visual mesh filename=package://hpp-rbprm-corba/meshes/ground_table.stl

File: data/urdf/stair_bauzil.urdf (robot description, URDF)
Before this commit: robot stair_bauzil, 1 links, 0 joints
Links:
- link base_link: geometry collision mesh filename=package://hpp-rbprm-corba/meshes/stair_bauzil_reduced.stl; visual mesh filename=package://hpp-rbprm-corba/meshes/stair_bauzil.stl
