Commit message: added truck scenario

File: data/urdf/car.urdf (robot description, URDF)
Before this commit: robot truck, 1 links, 0 joints
Links:
- link base_link: geometry collision mesh filename=package://hpp-rbprm-corba/meshes/car.stl; visual mesh filename=package://hpp-rbprm-corba/meshes/car.stl

File: data/urdf/hrp2_larm_rom.urdf (robot description, URDF)
Before this commit: robot hrp2_larm_rom, 4 links, 3 joints
Links:
- added link HEAD_LINK0, mass 0.374766
- added link HEAD_LINK1, mass 0.993355
Joints:
- added joint HEAD_JOINT0: type revolute, parent torso, child HEAD_LINK0, origin xyz=-0.007 0 0.2973 rpy=0 -0 0, axis 0 0 1, limit lower=-0.785398 upper=0.785398 effort=9.6 velocity=6.87679
- added joint HEAD_JOINT1: type revolute, parent HEAD_LINK0, child HEAD_LINK1, origin xyz=0 0 0 rpy=0 0 0, axis 0 1 0, limit lower=-0.523599 upper=0.785398 effort=9.6 velocity=6.87679

File: data/urdf/hrp2_lleg_rom.urdf (robot description, URDF)
Before this commit: robot hrp2_lleg_rom, 4 links, 3 joints
Links:
- added link HEAD_LINK0, mass 0.374766
- added link HEAD_LINK1, mass 0.993355
Joints:
- added joint HEAD_JOINT0: type revolute, parent torso, child HEAD_LINK0, origin xyz=-0.007 0 0.2973 rpy=0 -0 0, axis 0 0 1, limit lower=-0.785398 upper=0.785398 effort=9.6 velocity=6.87679
- added joint HEAD_JOINT1: type revolute, parent HEAD_LINK0, child HEAD_LINK1, origin xyz=0 0 0 rpy=0 0 0, axis 0 1 0, limit lower=-0.523599 upper=0.785398 effort=9.6 velocity=6.87679

File: data/urdf/hrp2_rarm_rom.urdf (robot description, URDF)
Before this commit: robot hrp2_rarm_rom, 4 links, 3 joints
Links:
- added link HEAD_LINK0, mass 0.374766
- added link HEAD_LINK1, mass 0.993355
Joints:
- added joint HEAD_JOINT0: type revolute, parent torso, child HEAD_LINK0, origin xyz=-0.007 0 0.2973 rpy=0 -0 0, axis 0 0 1, limit lower=-0.785398 upper=0.785398 effort=9.6 velocity=6.87679
- added joint HEAD_JOINT1: type revolute, parent HEAD_LINK0, child HEAD_LINK1, origin xyz=0 0 0 rpy=0 0 0, axis 0 1 0, limit lower=-0.523599 upper=0.785398 effort=9.6 velocity=6.87679

File: data/urdf/hrp2_rleg_rom.urdf (robot description, URDF)
Before this commit: robot hrp2_rleg_rom, 4 links, 3 joints
Links:
- added link HEAD_LINK0, mass 0.374766
- added link HEAD_LINK1, mass 0.993355
Joints:
- added joint HEAD_JOINT0: type revolute, parent torso, child HEAD_LINK0, origin xyz=-0.007 0 0.2973 rpy=0 -0 0, axis 0 0 1, limit lower=-0.785398 upper=0.785398 effort=9.6 velocity=6.87679
- added joint HEAD_JOINT1: type revolute, parent HEAD_LINK0, child HEAD_LINK1, origin xyz=0 0 0 rpy=0 0 0, axis 0 1 0, limit lower=-0.523599 upper=0.785398 effort=9.6 velocity=6.87679

File: data/urdf/hrp2_trunk_flexible.urdf (robot description, URDF)
Before this commit: robot hrp2_trunk_flexible, 4 links, 3 joints
Links:
- added link HEAD_LINK0, mass 0.374766; collision mesh filename=package://hrp2_14_description/meshes/convex/HEAD_LINK0.dae; visual mesh filename=package://hrp2_14_description/meshes/HEAD_LINK0.dae
- added link HEAD_LINK1, mass 0.993355; collision mesh filename=package://hrp2_14_description/meshes/convex/HEAD_LINK1.dae; visual mesh filename=package://hrp2_14_description/meshes/HEAD_LINK1.dae
Joints:
- added joint HEAD_JOINT0: type revolute, parent torso, child HEAD_LINK0, origin xyz=-0.007 0 0.2973 rpy=0 -0 0, axis 0 0 1, limit lower=-0.785398 upper=0.785398 effort=9.6 velocity=6.87679
- added joint HEAD_JOINT1: type revolute, parent HEAD_LINK0, child HEAD_LINK1, origin xyz=0 0 0 rpy=0 0 0, axis 0 1 0, limit lower=-0.523599 upper=0.785398 effort=9.6 velocity=6.87679
