Commit message: optimization

File: data/urdf/scene_wall2.urdf (robot description, URDF)
Before this commit: robot chair, 1 links, 0 joints
Links:
- link base_link: geometry collision mesh filename=package://hpp-rbprm-corba/meshes/ground_table2.stl; visual mesh filename=package://hpp-rbprm-corba/meshes/ground_table2.stl
