Commit message: added actual polaris mesh

File: data/urdf/polaris.urdf (robot description, URDF)
Before this commit: robot polaris, 1 links, 0 joints
Links:
- link base_link: geometry collision mesh filename=package://hpp-rbprm-corba/meshes/polaris.stl; visual mesh filename=package://hpp-rbprm-corba/meshes/polaris.stl
