Commit message: demo jump hyq work

File: data/urdf/ground_jump_easy.urdf (robot description, URDF)
Before this commit: robot ground_jump_easy, 3 links, 2 joints
Links:
- link groundStart: geometry collision mesh filename=package://hpp-rbprm-corba/meshes/ground_jump_easyStart2.stl; visual mesh filename=package://hpp-rbprm-corba/meshes/ground_jump_easyStart2.stl
