Commit message: down slope path work

File: data/urdf/downSlope.urdf (robot description, URDF)
Before this commit: robot hyq_trunk, 1 links, 0 joints
Links:
- link base_link: mass 50.26 -> None; geometry collision mesh filename=package://hpp-rbprm-corba/meshes/downSlope2.stl; visual mesh filename=package://hpp-rbprm-corba/meshes/downSlope2.stl
