Commit message: cleaning

File: data/urdf/hrp2_trunk_flexible.urdf (robot description, URDF)
Before this commit: robot hrp2_trunk_flexible, 4 links, 3 joints
Links:
- link BODY: geometry collision mesh filename=package://hpp-rbprm-corba/meshes/hrp2_trunk_body.stl; visual mesh filename=package://hpp-rbprm-corba/meshes/hrp2_lleg_rom.stl

Commit message: bug fixes on planning + new obstacle scene for hyq

File: data/urdf/hrp2_trunk_flexible.urdf (robot description, URDF)
Before this commit: robot hrp2_trunk_flexible, 4 links, 3 joints
Links:
- link BODY: geometry collision mesh filename=package://hpp-rbprm-corba/meshes/hrp2_trunk_body.stl; visual mesh filename=package://hpp-rbprm-corba/meshes/hrp2_trunk_body_view.dae
- link torso: geometry collision mesh filename=package://hpp-rbprm-corba/meshes/hrp2_trunk_torso.stl; visual mesh filename=package://hpp-rbprm-corba/meshes/hrp2_trunk_torso_view.dae

Commit message: downSlope path work, interp fail during transition slope/flat ground

File: data/urdf/hrp2_trunk_flexible.urdf (robot description, URDF)
Before this commit: robot hrp2_trunk_flexible, 6 links, 5 joints
Links:
- link BODY: mass None -> 58.0
- link HEAD_LINK0: mass 0.374766 -> None
- link HEAD_LINK1: mass 0.993355 -> None

File: data/urdf/hyq/hyq_trunk_large.urdf (robot description, URDF)
Before this commit: robot hyq_trunk_large, 1 links, 0 joints
Links:
- link base_link: geometry collision mesh filename=package://hpp-rbprm-corba/meshes/hyq/hyq_trunk_large3.stl; visual mesh filename=package://hpp-rbprm-corba/meshes/hyq/hyq_all.stl
