Commit message: add darpa meshs with reduced surface for hrp2 feet

File: data/urdf/darpa_no_ctc_mid.urdf (robot description, URDF)
Before this commit: robot chair, 1 links, 0 joints
Links:
- link base_link: geometry collision mesh filename=package://hpp-rbprm-corba/meshes/darpa_no_ctc_mid_collision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; visual mesh filename=package://hpp-rbprm-corba/meshes/darpa_no_ctc_mid.stl

Commit message: fix darpa mesh

File: data/urdf/darpa_no_ctc_mid.urdf (robot description, URDF)
Before this commit: robot chair, 1 links, 0 joints
Links:
- link base_link: geometry collision mesh filename=package://hpp-rbprm-corba/meshes/darpa_no_ctc_mid_collision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; visual mesh filename=package://hpp-rbprm-corba/meshes/darpa_no_ctc_mid_collision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
