Commit message: [demo] platform polytopes

File: data/urdf/cross_gap.urdf (robot description, URDF)
Before this commit: robot cross_gap, 1 links, 0 joints
Links:
- link base_link: geometry collision mesh filename=package://hpp-rbprm-corba/meshes/cross_gap2.stl; visual mesh filename=package://hpp-rbprm-corba/meshes/cross_gap2.stl
