Commit message: walk_bauzil scripts work

File: data/urdf/bauzil_stairs.urdf (robot description, URDF)
Before this commit: robot stair_bauzil, 1 links, 0 joints
Links:
- link base_link: geometry collision mesh filename=package://hpp-rbprm-corba/meshes/bauzil_walk_stairs.stl; visual mesh filename=package://hpp-rbprm-corba/meshes/bauzil_stairs.stl

Commit message: [meshes] update bauzil stairs meshs files to the new position of the stairs

File: data/urdf/bauzil_stairs.urdf (robot description, URDF)
Before this commit: robot stair_bauzil, 1 links, 0 joints
Links:
- link base_link: geometry collision mesh filename=package://hpp-rbprm-corba/meshes/bauzil_stairs_noRamp_simpl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; visual mesh filename=package://hpp-rbprm-corba/meshes/bauzil_stairs.stl
