Commit message: hyq model

File: data/urdf/hyq/hyq_trunk.urdf (robot description, URDF)
Before this commit: robot hyq_trunk, 1 links, 0 joints
Links:
- link base_link: geometry collision mesh filename=package://hpp-rbprm-corba/meshes/hyq/hyq_trunk.stl; visual mesh filename=package://hpp-rbprm-corba/meshes/hyq/hyq_all.stl
