Commit message: add mass information in HyQ urdf

File: data/urdf/hyq/hyq_trunk_large.urdf (robot description, URDF)
Before this commit: robot hyq_trunk_large, 1 links, 0 joints
Links:
- link base_link: mass None -> 50.26

Commit message: demo hrp2 downSlope work

File: data/urdf/hyq/hyq_trunk_large.urdf (robot description, URDF)
Before this commit: robot hyq_trunk_large, 1 links, 0 joints
Links:
- link base_link: geometry collision mesh filename=package://hpp-rbprm-corba/meshes/hyq/hyq_trunk_large2.stl scale=1 1 1; visual mesh filename=package://hpp-rbprm-corba/meshes/hyq/hyq_all.stl

Commit message: demo darpa work

File: data/urdf/hyq/hyq_trunk_large.urdf (robot description, URDF)
Before this commit: robot hyq_trunk_large, 1 links, 0 joints
Links:
- link base_link: geometry collision mesh filename=package://hpp-rbprm-corba/meshes/hyq/hyq_trunk_large.stl scale=1 1 1; visual mesh filename=package://hpp-rbprm-corba/meshes/hyq/hyq_all.stl

Commit message: darpa trunk large

File: data/urdf/hyq/hyq_trunk_large.urdf (robot description, URDF)
Before this commit: robot hyq_trunk_large, 1 links, 0 joints
Links:
- link base_link: geometry collision mesh filename=package://hpp-rbprm-corba/meshes/hyq/hyq_trunk_large4.stl scale=1 1 1; visual mesh filename=package://hpp-rbprm-corba/meshes/hyq/hyq_all.stl

Commit message: [urdf] fix hyq_trunk_large urdf

File: data/urdf/hyq/hyq_trunk_large.urdf (robot description, URDF)
Before this commit: robot hyq_trunk_large, 1 links, 0 joints
Links:
- link base_link: geometry collision mesh filename=package://hpp-rbprm-corba/meshes/hyq/hyq_trunk_large.stl; visual mesh filename=package://hpp-rbprm-corba/meshes/hyq/hyq_all.stl
