Commit message: window interpolation

File: data/urdf/siggraph_asia/wall.urdf (robot description, URDF)
Before this commit: robot wall, 1 links, 0 joints
Links:
- link base_link: geometry collision mesh filename=package://hpp-rbprm-corba/meshes/wall.stl; visual mesh filename=package://hpp-rbprm-corba/meshes/wall.stl
