Commit message: correcting configurations

File: data/spiderman/urdf/spiderman.urdf (robot description, URDF)
Before this commit: robot spiderman, 41 links, 40 joints
Joints:
- joint A_Skull_rx: limit lower=-0.3 upper=0.3 effort=0 velocity=1.0 -> lower=-0 upper=0 effort=0 velocity=1.0
- joint Skull_ry: limit lower=-1.1 upper=0.6 effort=0 velocity=1.0 -> lower=0 upper=0 effort=0 velocity=1.0
- joint Skull_rz: limit lower=-1.4 upper=1. effort=0 velocity=1.0 -> lower=-0 upper=0 effort=0 velocity=1.0
